File: pcb/_autosave-raspberry-flight-controller.kicad_sch (KiCad schematic)
At the start: 101 parts, among them J1 Conn_01x03, J10 Conn_02x20_Odd_Even, J11 Micro_SD_Card_Det1, J12 JTAG, J13 Conn_01x06, J14 Conn_01x06, J15 Conn_01x06, J16 Conn_01x06, J17 Conn_01x03, J18 Conn_01x03, J19 Conn_01x03, J2 Conn_01x03, J20 Conn_01x03, J21 Conn_01x06, J22 Conn_01x06, J3 Conn_01x03, J4 Conn_01x03, J5 Conn_01x03, J6 Conn_01x03, J8 Conn_02x05_Odd_Even, J9 POWER, SW1 SW_Push, SW2 SW_Push, SW3 SW_Push, SW4 SW_Push, U1 TPS54336ADRCR, U10 ISM330DHCX, U2 TPS54336ADRCR, U4 MIC5219-3.3YM5, U5 ISM330DHCX, U6 ISM330DHCX, U7 IST8310, U8 MS5611-01BA, U9 STM32F427VITx, Y1 Resonator

Commit message: Upload Files
Other:
- moved on the sheet: U10
Changed lines of the file:
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@@
 	(symbol
 		(lib_id "Sensor_Motion:ISM330DHCX")
-		(at 233.68 287.02 0)
+		(at 203.2 292.1 0)
 		(unit 1)
 		(exclude_from_sim no)
@@
 		(fields_autoplaced yes)
 		(property "Reference" "U10"
-			(at 235.8233 304.8 0)
+			(at 205.3433 309.88 0)
 			(effects
 				(font
@@
 		)
 		(property "Value" "ISM330DHCX"
-			(at 235.8233 307.34 0)
+			(at 205.3433 312.42 0)
 			(effects
 				(font
@@
 		)
 		(property "Footprint" "Package_LGA:LGA-14_3x2.5mm_P0.5mm_LayoutBorder3x4y"
-			(at 234.188 289.052 0)
+			(at 203.708 294.132 0)
 			(effects
 				(font
@@
 		)
 		(property "Datasheet" "https://www.st.com/resource/en/datasheet/ism330dhcx.pdf"
-			(at 234.442 288.798 0)
+			(at 203.962 293.878 0)
 			(effects
 				(font
@@
 		)
 		(property "Description" "iNEMO inertial module with embedded Machine Learning Core: always-on 3D accelerometer and 3D gyroscope with digital output for industrial applications, LGA-14"
-			(at 234.95 281.94 0)
+			(at 204.47 287.02 0)
 			(effects
 				(font
