File: pcb/raspberry-flight-controller.kicad_pcb (KiCad board)
At the start: 4 copper layers, 64 x 55 mm, 86 parts, among them J1 Conn_01x03, J2 Conn_01x03, J3 Conn_01x03, J4 Conn_01x03, J5 Conn_01x03, J6 Conn_01x03, J7 SWD, J8 Conn_02x05_Odd_Even, J9 POWER, SW1 SW_Push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

Commit message: Upload Files
Parts:
- removed J7: SWD, Connector_PinHeader_2.54mm:PinHeader_1x04_P2.54mm_Vertical
- removed U3: STM32F405RGTx, Package_QFP:LQFP-64_10x10mm_P0.5mm
- added C39: 100nF, Capacitor_SMD:C_0402_1005Metric, F.Cu at (121.2, 94.9)
- added C40: 100nF, Capacitor_SMD:C_0402_1005Metric, F.Cu at (121.2, 96.0)
- added J11: Micro_SD_Card_Det1, Connector_Card:microSD_HC_Molex_104031-0811, B.Cu at (147.8, 115.6)
- added J12: JTAG, Connector_JST:JST_SH_BM06B-SRSS-TB_1x06-1MP_P1.00mm_Vertical, F.Cu at (134.6, 76.9)
- added J13: Conn_01x06, Connector_JST:JST_SH_BM06B-SRSS-TB_1x06-1MP_P1.00mm_Vertical, F.Cu at (155.0, 78.0)
- added J14: Conn_01x06, Connector_JST:JST_SH_BM06B-SRSS-TB_1x06-1MP_P1.00mm_Vertical, F.Cu at (155.0, 85.0)
- added J15: Conn_01x06, Connector_JST:JST_SH_BM06B-SRSS-TB_1x06-1MP_P1.00mm_Vertical, F.Cu at (155.0, 92.0)
- added J16: Conn_01x06, Connector_JST:JST_SH_BM06B-SRSS-TB_1x06-1MP_P1.00mm_Vertical, F.Cu at (155.0, 99.0)
- added J17: Conn_01x03, Connector_PinHeader_2.54mm:PinHeader_1x03_P2.54mm_Vertical, F.Cu at (105.8, 93.2)
- added J18: Conn_01x03, Connector_PinHeader_2.54mm:PinHeader_1x03_P2.54mm_Vertical, F.Cu at (105.8, 95.8)
- added J19: Conn_01x03, Connector_PinHeader_2.54mm:PinHeader_1x03_P2.54mm_Vertical, F.Cu at (105.8, 98.3)
- added J20: Conn_01x03, Connector_PinHeader_2.54mm:PinHeader_1x03_P2.54mm_Vertical, F.Cu at (105.8, 100.9)
- added J21: Conn_01x06, Connector_JST:JST_SH_BM06B-SRSS-TB_1x06-1MP_P1.00mm_Vertical, F.Cu at (155.0, 106.0)
- added J22: Conn_01x06, Connector_JST:JST_SH_BM06B-SRSS-TB_1x06-1MP_P1.00mm_Vertical, F.Cu at (155.0, 113.0)
- added U10: ISM330DHCX, Package_LGA:LGA-14_3x2.5mm_P0.5mm_LayoutBorder3x4y, F.Cu at (120.0, 84.0)
- added U9: STM32F427VITx, Package_QFP:LQFP-100_14x14mm_P0.5mm, F.Cu at (131.0, 91.7)
- J1, J3, J5: footprint TiManh:Pad_PWM_Connector -> Connector_PinHeader_2.54mm:PinHeader_1x03_P2.54mm_Vertical
- J2, J4, J6: footprint TiManh:Pad_PWM_Connector -> Connector_PinHeader_2.54mm:PinHeader_1x03_P2.54mm_Vertical; moved to F.Cu
- moved C33 34.8 mm to (120.0, 81.7)
- moved C34 33.8 mm to (120.0, 86.4)
- moved SW2 30.4 mm to (146.7, 77.2), turned to -90 degrees
- moved C32 29.4 mm to (121.2, 93.8)
- moved SW1 28.5 mm to (142.4, 77.2), turned to -90 degrees
- moved R14 24.5 mm to (142.4, 80.5)
- moved C24 23.5 mm to (114.9, 99.5)
- moved C26 23.5 mm to (118.0, 102.0)
- moved C25 23.5 mm to (121.1, 99.5)
- moved U4 23.5 mm to (118.0, 99.5)
- moved R13 22.2 mm to (146.7, 80.5)
- moved U8 21.7 mm to (146.0, 89.0)
- moved C37 20.6 mm to (147.0, 113.3), turned to 180 degrees
- moved C12 19.8 mm to (128.9, 118.3)
- moved C19 19.8 mm to (130.8, 114.3)
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Routing:
- net +3.3VA: track 9.15 -> 0.00 mm
- net Net-(U9-VCAP_2): track 1.74 -> 0.00 mm
- net Net-(D6-A): track 0.00 -> 1.51 mm
- net Net-(D5-A): track 0.00 -> 1.51 mm
- net Net-(D2-A): track 0.00 -> 1.51 mm
- net Net-(D4-A): track 0.00 -> 1.49 mm
- net Net-(D3-A): track 0.00 -> 1.49 mm
- net Net-(D1-A): track 0.00 -> 1.49 mm
- net +5VP: vias 53 -> 35
- net GND: vias 102 -> 84
- removed copper zone on B.Cu, net +5VP
Other:
- outline, holes or cut-outs redrawn

Commit message: PCB update
Parts:
- added C41: 100nF, Capacitor_SMD:C_0603_1608Metric, F.Cu at (176.9, 99.0)
- moved J11 43.7 mm to (104.5, 109.8), turned to -90 degrees
- moved C25 5.27 mm to (117.1, 96.1), turned to 180 degrees
- moved C24 3.54 mm to (117.1, 102.3), turned to 0 degrees
- moved C26 3.22 mm to (119.5, 99.2), turned to 90 degrees
- moved U4 0.96 mm to (117.1, 99.2), turned to 90 degrees
Connections:
- U9 pad 25: unconnected-(U9-PA2-Pad25) -> USART2_TX
- U9 pad 26: unconnected-(U9-PA3-Pad26) -> USART2_RX
- U9 pad 30: unconnected-(U9-PA5-Pad30) -> SPI_SCK
- U9 pad 31: unconnected-(U9-PA6-Pad31) -> SPI_MISO
- U9 pad 32: unconnected-(U9-PA7-Pad32) -> SPI_MOSI
- U9 pad 38: unconnected-(U9-PE7-Pad38) -> UART7_RX
- U9 pad 39: unconnected-(U9-PE8-Pad39) -> UART7_TX
- U9 pad 47: unconnected-(U9-PB10-Pad47) -> USART3_TX
- U9 pad 48: unconnected-(U9-PB11-Pad48) -> USART3_RX
- U9 pad 78: unconnected-(U9-PC10-Pad78) -> USART4_TX
- U9 pad 79: unconnected-(U9-PC11-Pad79) -> USART4_RX
- U9 pad 92: unconnected-(U9-PB6-Pad92) -> I2C1_SCL
- U9 pad 93: unconnected-(U9-PB7-Pad93) -> I2C1_SDA
- U9 pad 97: unconnected-(U9-PE0-Pad97) -> USART8_RX
- U9 pad 98: unconnected-(U9-PE1-Pad98) -> USART8_TX
Routing:
- net +3.3VA: track 0.00 -> 21.9 mm, vias 0 -> 7
- net SWDIO: track 0.00 -> 10.9 mm
- net SWCLK: track 0.00 -> 6.17 mm, vias 0 -> 2
- net +5V: track 9.79 -> 15.4 mm
- net OSC_IN: track 0.00 -> 4.94 mm
- net OSC_OUT: track 0.00 -> 4.90 mm
- net Net-(U9-VCAP_2): track 0.00 -> 1.73 mm
- net Net-(U9-VCAP_1): track 0.00 -> 1.73 mm
- net Net-(U4-BP): track 0.00 -> 1.69 mm
- net Net-(C11-Pad1): track 0.00 -> 1.59 mm
