File: pcb/raspberry-flight-controller.kicad_pcb (KiCad board)
At the start: 4 copper layers, 64 x 55 mm, 101 parts, among them J1 Conn_01x03, J11 Micro_SD_Card_Det1, J12 JTAG, J13 Conn_01x06, J14 Conn_01x06, J15 Conn_01x06, J16 Conn_01x06, J17 Conn_01x03, J18 Conn_01x03, J19 Conn_01x03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

Commit message: update
Parts:
- added C42: 100nF, Capacitor_SMD:C_0603_1608Metric, F.Cu at (167.4, 89.8)
- added C43: 100nF, Capacitor_SMD:C_0603_1608Metric, F.Cu at (167.4, 92.3)
- added C44: 100nF, Capacitor_SMD:C_0603_1608Metric, F.Cu at (167.4, 94.8)
