File: pcb/raspberry-flight-controller.kicad_sch (KiCad schematic)
At the start: 101 parts, among them J1 Conn_01x03, J10 Conn_02x20_Odd_Even, J11 Micro_SD_Card_Det1, J12 JTAG, J13 Conn_01x06, J14 Conn_01x06, J15 Conn_01x06, J16 Conn_01x06, J17 Conn_01x03, J18 Conn_01x03, J19 Conn_01x03, J2 Conn_01x03, J20 Conn_01x03, J21 Conn_01x06, J22 Conn_01x06, J3 Conn_01x03, J4 Conn_01x03, J5 Conn_01x03, J6 Conn_01x03, J8 Conn_02x05_Odd_Even, J9 POWER, SW1 SW_Push, SW2 SW_Push, SW3 SW_Push, SW4 SW_Push, U1 TPS54336ADRCR, U10 ISM330DHCX, U2 TPS54336ADRCR, U4 MIC5219-3.3YM5, U5 ISM330DHCX, U6 ISM330DHCX, U7 IST8310, U8 MS5611-01BA, U9 STM32F427VITx, Y1 Resonator

Commit message: PCB update
Parts:
- added C41, C42, C43, C44: 100nF, Capacitor_SMD:C_0603_1608Metric, symbol Device:C
Connections:
- net I2C1_SCL: now also U9.92 (PB6)
- net I2C1_SDA: now also U9.93 (PB7)
- net SPI_MISO: now also U9.31 (PA6)
- net SPI_MOSI: now also U9.32 (PA7)
- net SPI_SCK: now also U9.30 (PA5)
- net UART7_RX: now also U9.38 (PE7)
- net UART7_TX: now also U9.39 (PE8)
- net USART3_RX: now also U9.48 (PB11)
- net USART3_TX: now also U9.47 (PB10)
- net USART4_RX: now also U9.79 (PC11)
- net USART4_TX: now also U9.78 (PC10)
- net USART2_TX: now reaches U9.25 (PA2)
- net USART2_RX: now reaches U9.26 (PA3)
- net USART8_RX: now reaches U9.97 (PE0)
- net USART8_TX: now reaches U9.98 (PE1)
Other:
- moved on the sheet: C1, C10, C11, C12, C13, C14, C15, C16, C17, C18, C19, C2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
